File: Laser_Electronics.kicad_pcb (KiCad board)
At the start: 2 copper layers, 36.8 x 90.2 mm, 43 parts, among them J1 MOT_X, J10 LIM_Y, J11 LED2, J2 GPIO, J3 UART, J4 LIM_X, J5 LASER, J6 POWER, J7 Micro_SD, J8 MOT_Y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

Commit message: UART reset circuit error repaired
Parts:
- R4, R5: value 1k -> 10k
Connections:
- J3 pad 2: /cts -> /rts
- J3 pad 6: /rts -> /dtr
- Q1 pad 2: /cts -> /rts
- Q1 pad 3: io00 -> /EN
- Q2 pad 2: /rts -> /dtr
- Q2 pad 3: /EN -> io00
- R4 pad 1: /rts -> /dtr
- R5 pad 1: /cts -> /rts
Routing:
- net /dtr: track 0.00 -> 49.9 mm, vias 0 -> 2
- net /cts: track 30.7 -> 0.00 mm, vias 2 -> 0
- net /rts: track 49.9 -> 30.7 mm
- net /EN: track 47.8 -> 54.6 mm
- net io00: track 87.0 -> 85.5 mm
- net DSBL: track 49.2 -> 48.5 mm
- net GND: vias 92 -> 103

Commit message: rev2 silkscreen + MiniLaser.yaml
Other:
- board text added: "rev 2"
- board text removed: "ver 1"
Changed lines of the file:
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@@
 		)
 	)
-	(gr_text "ver 1"
+	(gr_text "rev 2"
 		(at 120.142 73.406 0)
 		(layer "B.SilkS")
